Commit message: updated the world

File: my_robot/urdf/my_robot.xacro (robot description, xacro)
@@ -8,8 +8,8 @@
     </joint>
     <link name='chassis'>
-      <pose>0 0 0.1 0 0 0</pose>
+      <pose>0 0 0.075 0 0 0</pose> <!-- Updated Z position to half of the height -->
       <inertial>
         <mass value="15.0"/>
-        <origin xyz="0.0 0 0" rpy=" 0 0 0"/>
+        <origin xyz="0.0 0 0" rpy="0 0 0"/>
         <inertia
             ixx="0.1" ixy="0" ixz="0"
@@ -19,13 +19,13 @@
       </inertial>
       <collision name='collision'>
-        <origin xyz="0 0 0" rpy=" 0 0 0"/>
+        <origin xyz="0 0 0" rpy="0 0 0"/>
         <geometry>
-          <box size=".4 .2 .1"/>
+          <box size=".5 .3 .12"/> <!-- Updated chassis size -->
         </geometry>
       </collision>
       <visual name='chassis_visual'>
-        <origin xyz="0 0 0" rpy=" 0 0 0"/>
+        <origin xyz="0 0 0" rpy="0 0 0"/>
         <geometry>
-          <box size=".4 .2 .1"/>
+          <box size=".5 .3 .12"/> <!-- Updated chassis size -->
         </geometry>
         <material name="chassisMaterial">
@@ -34,146 +34,161 @@
       </visual>
       <collision name='back_caster_collision'>
-        <origin xyz="-0.15 0 -0.05" rpy=" 0 0 0"/>
+        <origin xyz="-0.15 0 -0.05" rpy="0 0 0"/>
         <geometry>
-          <sphere radius="0.0499"/>
+          <sphere radius="0.0999"/>
         </geometry>
       </collision>
       <visual name='back_caster_visual'>
-        <origin xyz="-0.15 0 -0.05" rpy=" 0 0 0"/>
+        <origin xyz="-0.15 0 -0.05" rpy="0 0 0"/>
         <geometry>
-          <sphere radius="0.05"/>
+          <sphere radius="0.10"/>
         </geometry>
       </visual>
       <collision name='front_caster_collision'>
-        <origin xyz="0.15 0 -0.05" rpy=" 0 0 0"/>
+        <origin xyz="0.15 0 -0.05" rpy="0 0 0"/>
         <geometry>
-          <sphere radius="0.0499"/>
+          <sphere radius="0.0999"/>
         </geometry>
       </collision>
       <visual name='front_caster_visual'>
-        <origin xyz="0.15 0 -0.05" rpy=" 0 0 0"/>
+        <origin xyz="0.15 0 -0.05" rpy="0 0 0"/>
         <geometry>
-          <sphere radius="0.05"/>
+          <sphere radius="0.10"/>
+        </geometry>
+      </visual>
+      <collision name='cylinder_head_collision'>
+        <origin xyz="-0.146012 0.0 0.1" rpy="0 0 0"/>
+        <geometry>
+          <cylinder radius="0.10" length="0.11"/>
+        </geometry>
+      </collision>
+      <visual name='cylinder_head_visual'>
+        <origin xyz="-0.146012 0.0 0.1" rpy="0 0 0"/>
+        <geometry>
+          <cylinder radius="0.10" length="0.11"/>
         </geometry>
       </visual>
     </link>
     <!-- Left Wheel -->
-  <link name="left_wheel">
-    <collision>
-      <geometry>
-        <cylinder radius="0.1" length="0.05"/>
-      </geometry>
-      <origin xyz="0 0 0" rpy="0 1.5707 1.5707"/>
-    </collision>
-    <inertial>
-      <mass value="5"/>
-      <inertia ixx="0.1" ixy="0" ixz="0" iyy="0.1" iyz="0" izz="0.1"/>
-    </inertial>
-    <visual name="left_wheel_visual">
-      <geometry>
-        <cylinder radius="0.1" length="0.05"/>
-      </geometry>
-      <material name="leftwheelMaterial">
-        <color rgba="1.0 0.0 0.0 1.0"/>
-      </material>
-      <origin xyz="0 0 0" rpy="0 1.5707 1.5707"/>
-    </visual>
-  </link>
-  <!-- Right Wheel -->
-  <link name="right_wheel">
-    <collision>
-      <geometry>
-        <cylinder radius="0.1" length="0.05"/>
-      </geometry>
-      <origin xyz="0 0 0" rpy="0 1.5707 1.5707"/>
-    </collision>
-    <inertial>
-      <mass value="5"/>
-      <inertia ixx="0.1" ixy="0" ixz="0" iyy="0.1" iyz="0" izz="0.1"/>
-    </inertial>
-    <visual name="right_wheel_visual">
-      <geometry>
-        <cylinder radius="0.1" length="0.05"/>
-      </geometry>
-      <material name="rightwheelMaterial">
-        <color rgba="1.0 0.0 0.0 1.0"/>
-      </material>
-      <origin xyz="0 0 0" rpy="0 1.5707 1.5707"/>
-    </visual>
-  </link>
-  <joint type="continuous" name="left_wheel_hinge">
-    <origin xyz="0 0.15 0" rpy="0 0 0"/>
-    <child link="left_wheel"/>
-    <parent link="chassis"/>
-    <axis xyz="0 1 0" rpy="0 0 0"/>
-    <limit effort="10000" velocity="1000"/>
-    <dynamics damping="1.0" friction="1.0"/>
-  </joint>
-  <joint type="continuous" name="right_wheel_hinge">
-    <origin xyz="0 -0.15 0" rpy="0 0 0"/>
-    <child link="right_wheel"/>
-    <parent link="chassis"/>
-    <axis xyz="0 1 0" rpy="0 0 0"/>
-    <limit effort="10000" velocity="1000"/>
-    <dynamics damping="1.0" friction="1.0"/>
-  </joint>
-  <!-- Camera -->
-  <link name="camera">
-    <collision>
-      <geometry>
-        <box size="0.05 0.05 0.05"/>
-      </geometry>
-      <origin xyz="0 0 0" rpy="0 0 0"/>
-    </collision>
-    <inertial>
-      <mass value="0.1"/>
-      <inertia ixx="1e-6" ixy="0" ixz="0" iyy="1e-6" iyz="0" izz="1e-6"/>
-    </inertial>
-    <visual name="camera_visual">
-      <geometry>
-        <box size="0.05 0.05 0.05"/>
-      </geometry>
-      <origin xyz="0 0 0" rpy="0 1.5707 1.5707"/>
-      <material name="CameraMaterial">
-        <color rgba="1.0 0.0 0.0 1.0"/>
-      </material>
-    </visual>
-   </link>
+    <link name="left_wheel">
+      <collision>
+        <geometry>
+          <cylinder radius="0.15" length="0.04"/> <!-- Updated radius -->
+        </geometry>
+        <origin xyz="0 0.05 0" rpy="0 1.5707 1.5707"/> <!-- Adjusted position -->
+      </collision>
+      <inertial>
+        <mass value="5"/>
+        <inertia ixx="0.1" ixy="0" ixz="0" iyy="0.1" iyz="0" izz="0.1"/>
+      </inertial>
+      <visual name="left_wheel_visual">
+        <geometry>
+          <cylinder radius="0.15" length="0.04"/> <!-- Updated radius -->
+        </geometry>
+        <material name="leftwheelMaterial">
+          <color rgba="1.0 0.0 0.0 1.0"/>
+        </material>
+        <origin xyz="0 0.05 0" rpy="0 1.5707 1.5707"/> <!-- Adjusted position -->
+      </visual>
+    </link>
+    <!-- Right Wheel -->
+    <link name="right_wheel">
+      <collision>
+        <geometry>
+          <cylinder radius="0.15" length="0.04"/> <!-- Updated radius -->
+        </geometry>
+        <origin xyz="0 -0.05 0" rpy="0 1.5707 1.5707"/> <!-- Adjusted position -->
+      </collision>
+      <inertial>
+        <mass value="5"/>
+        <inertia ixx="0.1" ixy="0" ixz="0" iyy="0.1" iyz="0" izz="0.1"/>
+      </inertial>
+      <visual name="right_wheel_visual">
+        <geometry>
+          <cylinder radius="0.15" length="0.04"/> <!-- Updated radius -->
+        </geometry>
+        <material name="rightwheelMaterial">
+          <color rgba="1.0 0.0 0.0 1.0"/>
+        </material>
+        <origin xyz="0 -0.05 0" rpy="0 1.5707 1.5707"/> <!-- Adjusted position -->
+      </visual>
+    </link>
+    <joint type="continuous" name="left_wheel_hinge">
+      <origin xyz="0 0.15 0" rpy="0 0 0"/>
+      <child link="left_wheel"/>
+      <parent link="chassis"/>
+      <axis xyz="0 1 0" rpy="0 0 0"/>
+      <limit effort="10000" velocity="1000"/>
+      <dynamics damping="1.0" friction="1.0"/>
+    </joint>
+    <joint type="continuous" name="right_wheel_hinge">
+      <origin xyz="0 -0.15 0" rpy="0 0 0"/>
+      <child link="right_wheel"/>
+      <parent link="chassis"/>
+      <axis xyz="0 1 0" rpy="0 0 0"/>
+      <limit effort="10000" velocity="1000"/>
+      <dynamics damping="1.0" friction="1.0"/>
+    </joint>
+    <!-- Camera -->
+    <link name="camera">
+      <collision>
+        <geometry>
+          <box size="0.05 0.02 0.02"/>
+        </geometry>
+        <origin xyz="0.03 0 -0.05" rpy="0 0 0"/>
+      </collision>
+      <inertial>
+        <mass value="0.1"/>
+        <inertia ixx="1e-6" ixy="0" ixz="0" iyy="1e-6" iyz="0" izz="1e-6"/>
+      </inertial>
+      <visual name="camera_visual">
+        <geometry>
+          <box size="0.05 0.02 0.02"/>
+        </geometry>
+        <origin xyz="0.03 0 -0.05" rpy="0 0 0"/>
+        <material name="CameraMaterial">
+          <color rgba="1.0 0.0 0.0 1.0"/>
+        </material>
+      </visual>
+    </link>
     <joint type="fixed" name="camera_joint">
-        <origin xyz="0.2 0 0" rpy="0 0 0"/>
+        <origin xyz="0.23 0 0.05" rpy="0 0 0"/> <!-- Updated Z position -->
         <child link="camera"/>
         <parent link="chassis"/>
     </joint>
     <gazebo reference="camera">
-        <material>Gazebo/Blue</material>
-      </gazebo>
-      <gazebo reference="chassis">
+        <material>Gazebo/Green</material>
+    </gazebo>
+    <gazebo reference="chassis">
         <material>Gazebo/Red</material>
-      </gazebo>
-      <gazebo reference="left_wheel">
-        <material>Gazebo/Green</material>
-      </gazebo>
-      <gazebo reference="right_wheel">
-        <material>Gazebo/Green</material>
-      </gazebo>
+    </gazebo>
+    <gazebo reference="cylinder_head">
+        <material>Gazebo/Red</material>
+    </gazebo>
+    <gazebo reference="left_wheel">
+        <material>Gazebo/Black</material>
+    </gazebo>
+    <gazebo reference="right_wheel">
+        <material>Gazebo/Black</material>
+    </gazebo>
     <!-- Lidar -->
-  <link name="hokuyo">
-    <collision>
-      <geometry>
-        <box size="0.1 0.1 0.1"/>
-      </geometry>
-      <origin xyz="0 0 0" rpy="0 0 0"/>
-    </collision>
-    <inertial>
-      <mass value="1e-5"/>
-      <inertia ixx="1e-6" ixy="0" ixz="0" iyy="1e-6" iyz="0" izz="1e-6"/>
-    </inertial>
-    <visual>
-      <geometry>
-        <mesh filename="package://my_robot/meshes/hokuyo.dae"/>
-      </geometry>
-      <origin xyz="0 0 0" rpy="0 0 0"/>
-    </visual>
-  </link>
+    <link name="hokuyo">
+      <collision>
+        <geometry>
+          <box size="0.1 0.1 0.1"/>
+        </geometry>
+        <origin xyz="0 0 0" rpy="0 0 0"/>
+      </collision>
+      <inertial>
+        <mass value="1e-5"/>
+        <inertia ixx="1e-6" ixy="0" ixz="0" iyy="1e-6" iyz="0" izz="1e-6"/>
+      </inertial>
+      <visual>
+        <geometry>
+          <mesh filename="package://my_robot/meshes/hokuyo.dae"/>
+        </geometry>
+        <origin xyz="0 0 0" rpy="0 0 0"/>
+      </visual>
+    </link>
     <joint type="fixed" name="hokuyo_joint">
         <origin xyz="0.15 0 0.1" rpy="0 0 0"/>
@@ -181,3 +196,3 @@
         <parent link="chassis"/>
     </joint>
-  </robot>
+</robot>
